File: cir/BD/BD.kicad_pcb (KiCad board)
At the start: 4 copper layers, 11 parts, among them J1 Conn_01x06_Socket, J2 Conn_01x04_Socket, J3 Conn_01x02_Socket, SW1 SW_Push, SW2 SW_Push

Commit message: uo
Parts:
- moved R1 43.2 mm to (20.3, 42.5), turned to 90 degrees
- moved R2 40.6 mm to (24.4, 42.5), turned to 90 degrees
- moved J3 39.6 mm to (21.0, 57.1)
- moved J1 35.6 mm to (28.4, 17.7), turned to -90 degrees
- moved D1 31.3 mm to (24.3, 34.4)
- moved D2 30.6 mm to (18.5, 34.7)
- moved SW2 30.3 mm to (19.8, 27.3), turned to -90 degrees
- moved SW1 27.8 mm to (26.2, 27.3), turned to -90 degrees
- moved J2 27.1 mm to (18.4, 59.7), turned to 90 degrees
- moved A1 2.61 mm to (30.0, 23.5)
- moved U1 1.89 mm to (22.4, 47.6)
Routing:
- net GND: track 0.00 -> 57.3 mm
- net VCC: track 0.00 -> 45.9 mm
- net Net-(A1-A0): track 0.02 -> 40.1 mm
- net Net-(A1-A1): track 0.00 -> 36.7 mm
- net Net-(A1-A2): track 0.00 -> 33.6 mm
- net Net-(A1-A3): track 0.00 -> 30.5 mm, vias 0 -> 2
- net +5V: track 0.00 -> 28.3 mm, vias 0 -> 1
- net Net-(A1-SDA/A4): track 0.00 -> 24.3 mm
- net Net-(A1-SCL/A5): track 0.00 -> 22.3 mm, vias 0 -> 1
- net Net-(J2-Pin_4): track 0.00 -> 18.9 mm
- net SW1: track 0.00 -> 18.1 mm, vias 0 -> 1
- net Net-(J2-Pin_3): track 0.00 -> 17.1 mm
- net SW2: track 0.00 -> 17.0 mm, vias 0 -> 1
- net Net-(J2-Pin_2): track 0.00 -> 12.3 mm
- net Net-(A1-D4): track 0.00 -> 10.5 mm
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Other:
- board outline added: 18.3 x 52.8 mm
