File: cir/BD/BD.kicad_pcb (KiCad board)
At the start: 2 copper layers, 21.6 x 57.6 mm, 11 parts, among them J1 Conn_01x06_Socket, J2 Conn_01x04_Socket, J4 Barrel_Jack_MountingPin, SW1 SW_Push, SW2 SW_Push

Commit message: uo
Parts:
- A1, J4: moved to F.Cu
- SW2: moved to B.Cu
- moved J1 75.3 mm to (100.3, 54.6)
- moved SW1 74.4 mm to (108.0, 45.7), turned to 90 degrees
- moved SW2 68.5 mm to (108.0, 30.5)
- moved R2 67.9 mm to (102.9, 31.8), turned to -90 degrees
- moved R1 65.4 mm to (100.3, 34.3), turned to -90 degrees
- moved J4 52.8 mm to (88.6, 20.0)
- moved D1 45.9 mm to (74.9, 36.8)
- moved A1 39.0 mm to (81.3, 26.7), turned to 0 degrees
- moved D2 37.5 mm to (74.9, 41.9)
- moved J2 33.9 mm to (58.4, 55.9), turned to 180 degrees
- moved U1 33.6 mm to (67.3, 52.1)
Routing:
- net VCC: track 53.5 -> 0.00 mm
- net +5V: track 32.9 -> 0.00 mm
- net Net-(J2-Pin_4): track 19.6 -> 0.00 mm
- net SW2: track 18.9 -> 0.00 mm, vias 2 -> 0
- net GND: track 17.6 -> 0.00 mm, vias 8 -> 0
- net Net-(J2-Pin_3): track 16.0 -> 0.00 mm
- net Net-(A1-D2): track 15.8 -> 0.00 mm, vias 3 -> 0
- net Net-(J2-Pin_2): track 12.4 -> 0.00 mm
- net Net-(J2-Pin_1): track 9.62 -> 0.00 mm
- net SW1: track 8.48 -> 0.00 mm
- net IN3: track 3.59 -> 0.00 mm
- net IN2: track 3.59 -> 0.00 mm
- net IN1: track 3.59 -> 0.00 mm
- net IN4: track 3.59 -> 0.00 mm
- net Net-(A1-SDA/A4): track 3.05 -> 0.00 mm
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- removed copper zone on B.Cu, net GND
Other:
- board outline removed
