File: cir/LT/LT.kicad_sch (KiCad schematic)
At the start: 22 parts, among them J1 Conn_01x04_Socket, U1 LBR-127HLD, U2 74HC7014, U4 LBR-127HLD, U5 LBR-127HLD, U6 LBR-127HLD

Commit message: rr
Parts:
- added J2: Conn_01x04_Socket, Connector_PinHeader_2.54mm:PinHeader_1x04_P2.54mm_Vertical, symbol Connector:Conn_01x04_Socket
- added J3: Conn_01x02_Socket, Connector_PinHeader_2.54mm:PinHeader_1x02_P2.54mm_Vertical, symbol Connector:Conn_01x02_Socket
- D1, D2, D3, D4: footprint LED_THT:LED_BL-FL7680RGB -> LED_THT:LED_D3.0mm
- R2, R4, R7, R8: footprint (none) -> 自作:R_Variable
Connections:
- net +5V: now also J3.1 (Pin_1)
- net GND: now also J3.2 (Pin_2)
- net S1: now also U2.13; no longer U2.1
- net S2: now also U2.9; no longer U2.3
- net S3: now also U2.11; no longer U2.9
- net S4: now also U2.5; no longer U2.11
- net at D2.2 (A): now also U2.8; no longer U2.4
- net at U2.2: now also J2.2 (Pin_2); no longer D1.2 (A)
- net at D3.2 (A): now also U2.10; no longer U2.8
- net at D4.2 (A): now also U2.6; no longer U2.10
- net at U2.12: now also D1.2 (A)
- new net: J2.1 (Pin_1), U2.1
- new net: J2.3 (Pin_3), U2.3
- new net: J2.4 (Pin_4), U2.4
Other:
- moved on the sheet: U2A, U2B, U2C, U2D, U2E, U2F

Commit message: uo
Connections:
- net S1: now also U2.1; no longer U2.13
- net S2: now also U2.5; no longer U2.9
- net S4: now also U2.9; no longer U2.5
- net at D2.2 (A): now also U2.6; no longer U2.8
- net at J2.1 (Pin_1): now also U2.4; no longer U2.1
- net at J2.2 (Pin_2): now also U2.3; no longer U2.2
- net at J2.3 (Pin_3): now also U2.12; no longer U2.3
- net at J2.4 (Pin_4): now also U2.13; no longer U2.4
- net at D1.2 (A): now also U2.2; no longer U2.12
- net at D4.2 (A): now also U2.8; no longer U2.6
Other:
- moved on the sheet: U2A, U2B, U2C, U2D, U2F

Commit message: u
Parts:
- R1, R10, R11, R12, R3, R5, R6, R9: footprint Resistor_SMD:R_2010_5025Metric -> Resistor_THT:R_Axial_DIN0204_L3.6mm_D1.6mm_P5.08mm_Horizontal
- U2: footprint Package_SO:SOIC-14_3.9x8.7mm_P1.27mm -> Package_DIP:DIP-14_W7.62mm_Socket
Connections:
- net at D2.2 (A): now also U2.12; no longer U2.6
- net at J2.1 (Pin_1): now also U2.3; no longer U2.4
- net at J2.2 (Pin_2): now also U2.4; no longer U2.3
- net at J2.3 (Pin_3): now also U2.5; no longer U2.12
- net at J2.4 (Pin_4): now also U2.6; no longer U2.13
- net S1: no longer names the net of J1.1 (Pin_1), R2.1, U1.4 (Collector), U2.1
- net S2: no longer names the net of J1.2 (Pin_2), R4.1, U4.4 (Collector)
- net S2: now also U2.13; no longer U2.5
- net S3: no longer names the net of J1.3 (Pin_3), R7.1, U2.11, U5.4 (Collector)
- net S4: no longer names the net of J1.4 (Pin_4), R8.1, U2.9, U6.4 (Collector)
Other:
- moved on the sheet: D1, D2, D3, D4, J1, J2, J3, R1, R10, R11, R12, R2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

Commit message: up
Parts:
- J1: value Conn_01x04_Socket -> Arduino
- J3: value Conn_01x02_Socket -> Power
Connections:
- net at R4.1, U2.13, U4.4 (Collector): now also J1.4 (Pin_4); no longer J1.2 (Pin_2)
- net at R7.1, U2.11, U5.4 (Collector): now also J1.2 (Pin_2); no longer J1.3 (Pin_3)
- net at R8.1, U2.9, U6.4 (Collector): now also J1.3 (Pin_3); no longer J1.4 (Pin_4)
Other:
- moved on the sheet: D1, D2, D3, D4, J1, J2, J3, R1, R10, R11, R12, R2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
