File: cir/ultra_seigyo/ultra_seigyo.kicad_pcb (KiCad board)
At the start: 4 copper layers, 30 parts, among them IC1 tc74hc21ap, IC2 tc74hc21ap, J1 Conn_01x04_Socket, J2 Conn_01x02_Pin, J3 Conn_01x02_Pin, U1 74LS07, U10 NJM4558, U11 NJM4558, U12 NMA0515SC, U2 74HC74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

Commit message: uo
Parts:
- removed RV1: R_Potentiometer, Potentiometer_THT:Potentiometer_Bourns_3296X_Horizontal
- removed U2: 74HC74, Package_DIP:DIP-14_W7.62mm_Socket
- removed U3: ~, Package_DIP:DIP-8_W7.62mm_Socket
- moved J3 98.8 mm to (121.9, 101.6), turned to 0 degrees
- moved J2 95.1 mm to (109.2, 111.8), turned to 180 degrees
- moved U12 92.4 mm to (100.0, 111.7), turned to 180 degrees
- moved R8 89.5 mm to (86.4, 129.5)
- moved U8 88.4 mm to (38.1, 121.9), turned to 90 degrees
- moved R7 81.9 mm to (86.4, 127.0)
- moved U6 81.8 mm to (101.6, 50.8), turned to -90 degrees
- moved R1 81.6 mm to (91.4, 124.5)
- moved R5 81.4 mm to (94.0, 119.4)
- moved U10 81.4 mm to (94.0, 121.9)
- moved R3 81.3 mm to (104.1, 129.5)
- moved RV4 71.2 mm to (109.2, 119.4), turned to 90 degrees
- moved U7 66.2 mm to (58.4, 121.9), turned to 90 degrees
- moved R9 65.9 mm to (106.7, 73.7), turned to -90 degrees
- moved U5 64.8 mm to (58.4, 61.0), turned to 90 degrees
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Connections:
- U1 pad 10: B -> A
- U1 pad 11: Net-(J1-Pin_2) -> Net-(J1-Pin_1)
- U1 pad 12: unconnected-(U1-Pad12) -> B
- U1 pad 13: unconnected-(U1-Pad13) -> Net-(J1-Pin_2)
- U1 pad 8: A -> unconnected-(U1-Pad8)
- U1 pad 9: Net-(J1-Pin_1) -> unconnected-(U1-Pad9)
- U4 pad 10: ~B -> ~A
- U4 pad 11: B -> A
- U4 pad 12: unconnected-(U4-Pad12) -> ~B
- U4 pad 13: unconnected-(U4-Pad13) -> B
- U4 pad 5: unconnected-(U4-Pad5) -> F
- U4 pad 6: unconnected-(U4-Pad6) -> ~F
- U4 pad 8: ~A -> ~E
- U4 pad 9: A -> E
- U9 pad 1: D_1 -> E
- U9 pad 4: D_2 -> F
Routing:
- net +5V: track 563.9 -> 352.9 mm, vias 9 -> 11
- net GND: track 482.6 -> 271.8 mm, vias 13 -> 16
- net -5V: track 266.8 -> 60.0 mm
- net ML0: track 5.08 -> 129.1 mm, vias 0 -> 2
- net ~E: track 236.2 -> 123.0 mm, vias 0 -> 3
- net ~F: track 209.9 -> 105.8 mm, vias 0 -> 4
- net ML1: track 2.54 -> 99.2 mm, vias 0 -> 1
- net B: track 147.3 -> 242.1 mm
- net D: track 97.6 -> 165.1 mm
- net ~A: track 139.3 -> 78.3 mm, vias 7 -> 3
- net ~D: track 106.7 -> 46.8 mm, vias 4 -> 2
- net Net-(IC2-Pad8): track 12.3 -> 68.6 mm, vias 0 -> 2
- net Net-(IC1-Pad8): track 15.2 -> 68.6 mm, vias 0 -> 2
- net F: track 83.8 -> 41.7 mm, vias 2 -> 0
- net Net-(U5-Pad6): track 71.1 -> 32.1 mm, vias 0 -> 2
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