File: cir/ultra_seigyo/ultra_seigyo.kicad_sch (KiCad schematic)
At the start: 14 parts, among them IC1 tc74hc21ap, IC2 tc74hc21ap, J1 Conn_01x04_Socket, U1 74LS07, U10 NJM4558, U2 74HC74, U4 74HC04, U5 74HC00, U6 74HC02, U7 74HC00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

Commit message: ki
Parts:
- added J2, J3: Conn_01x02_Pin, Connector_PinSocket_2.54mm:PinSocket_1x02_P2.54mm_Vertical, symbol Connector:Conn_01x02_Pin
- added R1, R2: 5.1k, Resistor_THT:R_Axial_DIN0204_L3.6mm_D1.6mm_P5.08mm_Horizontal, symbol Device:R
- added R10, R3, R4, R5, R6, R7, R8, R9: 10k, Resistor_THT:R_Axial_DIN0204_L3.6mm_D1.6mm_P5.08mm_Horizontal, symbol Device:R
- added RV4, RV5: R_Potentiometer, Potentiometer_THT:Potentiometer_Bourns_3296X_Horizontal, symbol Device:R_Potentiometer
- added U11: NJM4558, Package_DIP:DIP-8_W7.62mm_Socket, symbol Amplifier_Operational:NJM4558
- added U12: NMA0515SC, Converter_DCDC:Converter_DCDC_Murata_NMAxxxxSC_THT, symbol Regulator_Switching:NMA0515SC
- added unit 3 of U4
- IC1, IC2: footprint DIP14 -> Package_DIP:DIP-14_W7.62mm_Socket
- U3: footprint (none) -> Package_DIP:DIP-8_W7.62mm_Socket
- U4, U6, U9: footprint (none) -> Package_DIP:DIP-14_W7.62mm_Socket
Connections:
- net D~ is gone; now on net ~D: U7.2
- net +5V: now also U10.8 (V+), J3.1 (Pin_1), U11.8 (V+), U12.6 (VOUT+)
- net A: now also U1.8, U4.9; no longer U1.2, U4.1
- net B: now also U1.10, U4.11; no longer U1.4, U4.3
- net C: now also U1.2, U4.1; no longer U1.6, U4.5
- net CLR: now also U3.8 (OUT); no longer U3.5 (OUT)
- net D: now also U1.4, U4.3; no longer U1.8, U4.9
- net E: now also IC1.4; no longer IC1.5
- net F: now also IC2.4; no longer IC2.5
- net GND: now also U3.5 (GND), J3.2 (Pin_2), RV4.1, RV5.1, U12.5 (0V); no longer U3.8 (GND)
- net MR0: now also R9.1; no longer U8.10, U8.11
- net MR1: now also R10.1; no longer U8.13
- net ~A: now also U4.8; no longer U4.2
- net ~B: now also IC2.10, U4.10; no longer IC2.9, U4.4
- net ~C: now also IC1.5, U4.2; no longer IC1.4, U4.6
- net ~D: now also IC2.5, IC2.9, U4.4; no longer IC2.10, IC2.4, U4.8
- net at U10.5 (+): now also R5.2
- net at U10.6 (-): now also R3.1
- net at U10.7: now also R3.2, RV4.3
- net at J1.1 (Pin_1): now also U1.9; no longer U1.1
- net at J1.2 (Pin_2): now also U1.11; no longer U1.3
- net at J1.3 (Pin_3): now also U1.1; no longer U1.5
- net at J1.4 (Pin_4): now also U1.3; no longer U1.9
- net -5V: now reaches U10.4 (V-)
- net -5V: now also U11.4 (V-), U12.4 (VOUT-)
- net at U10.1: now also R1.2, R5.1
- net at U10.2 (-): now also R1.1
- net at U10.3 (+): now also R7.2, R8.2
- new net: R4.2, RV5.3, U11.7
- new net: R10.2, R9.2, U11.3 (+)
- new net: R4.1, U11.6 (-)
- new net: R2.2, R6.1, U11.1
- new net: R6.2, U11.5 (+)
- new net: R2.1, U11.2 (-)
- new net: J2.1 (Pin_1), U12.1 (VIN+)
- new net: J2.2 (Pin_2), U12.2 (VIN-)
- new net MD_IN1: RV4.2
- new net MD_IN2: RV5.2
- new net ML0: R7.1, U8.10, U8.11
- new net ML1: R8.1, U8.13
Other:
- moved on the sheet: U10A, U10B, U10C, U1A, U1C

Commit message: uo
Parts:
- removed RV1: R_Potentiometer, Potentiometer_THT:Potentiometer_Bourns_3296X_Horizontal, symbol Device:R_Potentiometer
- removed U2: 74HC74, Package_DIP:DIP-14_W7.62mm_Socket, symbol 74xx:74HC74
- removed U3: ~, Package_DIP:DIP-8_W7.62mm_Socket, symbol 自作:LTC1799
Connections:
- net D_1 is gone; now on net E: U9.1
- net D_2 is gone; now on net F: U9.4
- net A: now also U1.10, U4.11; no longer U1.8, U4.9
- net B: now also U1.12, U4.13; no longer U1.10, U4.11
- net E: now also U4.9
- net F: now also U4.5
- net ~A: now also U4.10; no longer U4.8
- net ~B: now also U4.12; no longer U4.10
- net ~E: now also U4.8
- net ~F: now also U4.6
- net at J1.1 (Pin_1): now also U1.11; no longer U1.9
- net at J1.2 (Pin_2): now also U1.13; no longer U1.11
Other:
- moved on the sheet: U4C, U4D
