File: cir/trss2/trss2.kicad_pcb (KiCad board)
At the start: 2 copper layers, 184.2 x 139.7 mm, 108 parts, among them J1 Conn_01x04_Socket, J10 Conn_01x06_Socket, J11 Conn_01x06_Socket, J2 Conn_01x02_Socket, J3 Conn_01x02_Socket, J4 Conn_01x02_Socket, J6 Conn_01x02_Socket, J7 Conn_01x06_Socket, J8 Conn_01x06_Socket, J9 Conn_01x03_Socket, Q1 2SC1815, Q10 2SC1815, Q11 2SC1815, Q12 2SC1815, Q13 2SC1815, Q14 2SC1815, Q15 2SC1815, Q16 2SC1815, Q17 2SC1815, Q18 2SC1815, Q19 2SC1815, Q2 2SC1815, Q20 2SC1815, Q21 2SC1815, Q22 2SC1815, Q23 2SC1815, Q24 2SC1815, Q25 2SC1815, Q26 2SC1815, Q27 2SC1815, Q28 2SC1815, Q29 2SC1815, Q3 2SC1815, Q30 2SC1815, Q31 2SC1815, Q32 2SC1815, Q33 2SC1815, Q34 2SC1815, Q35 2SC1815, Q36 2SC1815, Q37 2SC1815, Q38 2SC1815, Q39 2SC1815, Q4 2SC1815, Q40 2SC1815, Q5 2SC1815, Q6 2SC1815, Q7 2SC1815, Q8 2SC1815, Q9 2SC1815, U1 NJM4558, U2 NJM4558, U3 NMA0515SC

Commit message: go
Parts:
- added J10: Conn_01x06_Socket, Connector_PinSocket_2.54mm:PinSocket_1x06_P2.54mm_Vertical, F.Cu at (200.7, 101.6)
- moved Q16 19.1 mm to (243.8, 96.5)
- moved Q23 19.1 mm to (243.8, 114.3)
- moved R33 19.0 mm to (248.9, 104.1)
- moved R34 19.0 mm to (248.9, 116.8)
- moved Q11 16.5 mm to (251.5, 137.2)
- moved Q24 16.5 mm to (241.3, 132.1)
- moved R22 16.5 mm to (251.5, 147.3)
- moved R27 16.5 mm to (233.7, 91.4)
- moved Q10 16.5 mm to (248.9, 142.2)
- moved Q14 16.5 mm to (231.1, 142.2)
- moved Q15 16.5 mm to (228.6, 132.1)
- moved Q17 16.5 mm to (236.2, 94.0)
- moved Q18 16.5 mm to (231.1, 91.4)
- moved Q21 16.5 mm to (231.1, 127.0)
- moved Q22 16.5 mm to (228.6, 137.2)
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Routing:
- net C_~C: track 63.1 -> 104.1 mm, vias 2 -> 6
- net C_~B: track 78.5 -> 116.8 mm, vias 4 -> 8
- net C_~B~DF: track 37.7 -> 65.6 mm, vias 3 -> 2
- net C_~E~F: track 40.2 -> 66.0 mm, vias 2 -> 4
- net C_D: track 25.4 -> 40.6 mm, vias 0 -> 2
- net C_A: track 12.7 -> 27.9 mm
- net C_~D: track 34.1 -> 49.3 mm
- net C_~A: track 71.7 -> 84.9 mm, vias 2 -> 4
- net +5V: track 433.9 -> 430.1 mm
- net Net-(Q16-E): track 5.08 -> 7.62 mm
- net C_F: track 12.7 -> 15.2 mm
- net MR0: track 29.0 -> 30.5 mm
- net Net-(Q23-E): track 23.9 -> 22.9 mm
- net Net-(Q32-E): track 5.08 -> 6.13 mm
- net GND: vias 12 -> 13
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Other:
- board size 184.2 x 139.7 mm -> 190.5 x 139.7 mm

Commit message: >
Parts:
- moved R28 15.5 mm to (210.8, 94.0), turned to 0 degrees
- moved Q39 10.2 mm to (218.4, 109.2)
- moved Q40 10.2 mm to (221.0, 104.1)
- moved Q16 8.03 mm to (236.2, 99.1)
- moved R27 8.03 mm to (226.1, 94.0)
- moved Q17 8.03 mm to (228.6, 96.5)
- moved Q18 8.03 mm to (223.5, 94.0)
- moved Q11 7.62 mm to (243.8, 137.2)
- moved Q15 7.62 mm to (221.0, 132.1)
- moved Q22 7.62 mm to (221.0, 137.2)
- moved Q23 7.62 mm to (236.2, 114.3)
- moved Q24 7.62 mm to (233.7, 132.1)
- moved Q32 7.62 mm to (218.4, 114.3)
- moved Q9 7.62 mm to (238.8, 147.3)
- moved R21 7.62 mm to (246.4, 142.2)
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Routing:
- net C_~C: track 104.1 -> 78.7 mm, vias 6 -> 4
- net C_~B: track 116.8 -> 99.1 mm, vias 8 -> 7
- net C_~D: track 49.3 -> 36.6 mm
- net C_A: track 27.9 -> 17.8 mm
- net C_~A~CE: track 66.0 -> 58.4 mm
- net C_~A: track 84.9 -> 77.3 mm
- net C_D: track 40.6 -> 33.0 mm
- net C_~E~F: track 66.0 -> 58.4 mm
- net C_~B~DF: track 65.6 -> 58.4 mm, vias 2 -> 3
- net Net-(Q36-E): track 15.2 -> 20.3 mm
- net GND: track 369.6 -> 367.1 mm, vias 13 -> 12
- net C_F: track 15.2 -> 12.7 mm
- net Net-(Q18-E): track 7.62 -> 10.2 mm
