File: cir/trss3/trss3.kicad_sch (KiCad schematic)
At the start: 51 parts, among them J1 Conn_01x04, Q1 2SC1815, Q10 2SC1815, Q11 2SA1015, Q12 2SA1015, Q13 2SA1015, Q14 2SC1815, Q15 2SC1815, Q16 2SC1815, Q17 2SA1015, Q18 2SA1015, Q19 2SA1015, Q2 2SA1015, Q20 2SC1815, Q21 2SC1815, Q22 2SC1815, Q23 2SA1015, Q24 2SC1815, Q25 2SC1815, Q26 2SA1015, Q27 2SC1815, Q28 2SA1015, Q29 2SC1815, Q3 2SA1015, Q30 2SA1015, Q31 2SA1015, Q32 2SC1815, Q4 2SC1815, Q5 2SA1015, Q6 2SA1015, Q7 2SA1015, Q8 2SC1815, Q9 2SC1815, U1 OKI-78SR-12_1.0-W36-C, U2 74LS07

Commit message: up
Parts:
- removed R10, R11, R12, R9: 5.1k, symbol Device:R
- removed U2: 74LS07, Package_DIP:DIP-14_W7.62mm_Socket, symbol 74xx:74LS07
- added Q33, Q34, Q35, Q36, Q37, Q38, Q39, Q40: 2SC1815, Package_TO_SOT_THT:TO-92L_Inline_Wide, symbol Transistor_BJT:2SC1815
- added R17, R22, R25, R28: 27k, Resistor_THT:R_Axial_DIN0204_L3.6mm_D1.6mm_P5.08mm_Horizontal, symbol Device:R
- added R18, R20, R23, R26: 10k, Resistor_THT:R_Axial_DIN0204_L3.6mm_D1.6mm_P5.08mm_Horizontal, symbol Device:R
- added R19, R21, R24, R27: 4.6k, Resistor_THT:R_Axial_DIN0204_L3.6mm_D1.6mm_P5.08mm_Horizontal, symbol Device:R
- R13, R14, R15, R16: footprint (none) -> Resistor_THT:R_Axial_DIN0204_L3.6mm_D1.6mm_P5.08mm_Horizontal
Connections:
- net MR is gone; now on net MR0: Q16.1 (E), Q18.1 (E), Q20.1 (E), Q21.1 (E), R5.1
- net +5V: now also R17.1, R18.1, R20.1, R22.1, R23.1, R25.1, R26.1, R28.1
- net A: now also Q34.2 (C), R17.2
- net A_IN: now also Q33.3 (B)
- net B: now also Q36.2 (C), R22.2
- net B_IN: now also Q35.3 (B)
- net C: now also Q38.2 (C), R25.2
- net C_IN: now also Q37.3 (B)
- net D: now also Q40.2 (C), R28.2
- net D_IN: now also Q39.3 (B)
- net GND: now also Q34.1 (E), Q36.1 (E), Q38.1 (E), Q40.1 (E), R19.2, R21.2, R24.2, R27.2
- new net: Q33.2 (C), Q34.3 (B), R18.2
- new net: Q33.1 (E), R19.1
- new net: Q35.2 (C), Q36.3 (B), R20.2
- new net: Q39.2 (C), Q40.3 (B), R26.2
- new net: Q35.1 (E), R21.1
- new net: Q37.2 (C), Q38.3 (B), R23.2
- new net: Q39.1 (E), R27.1
- new net: Q37.1 (E), R24.1
